File: 68uino/68uino.kicad_sch (KiCad schematic)
At the start: 24 parts, among them SW1 SW_Push, U1 HD6303, U2 27C256, U4 74LS373, U5 NE555P

Commit message: update
Parts:
- removed R3: 5k, Resistor_THT:R_Axial_DIN0207_L6.3mm_D2.5mm_P7.62mm_Horizontal, symbol Device:R
- removed U2: 27C256, Package_DIP:DIP-28_W15.24mm, symbol Memory_EPROM:27C256
- removed U5: NE555P, Package_DIP:DIP-8_W7.62mm, symbol Timer:NE555P
- added C10, C11, C7, C8, C9: 1uF, Capacitor_THT:C_Disc_D6.0mm_W2.5mm_P5.00mm, symbol Device:C_Small
- added J1: P/S 2 Breakout, Custom_Footprints:Connector_Mini-DIN_Female_6Pin_2rows, symbol Connector:Mini-DIN-6
- added J2: R232 Plug, Connector_Dsub:DSUB-9_Female_Horizontal_P2.77x2.84mm_EdgePinOffset9.90mm_Housed_MountingHolesOffset11.32mm, symbol Connector:DE9_Plug
- added J3: Screen, symbol Connector:Conn_01x04_Pin
- added R3, R9: 1k, Resistor_THT:R_Axial_DIN0207_L6.3mm_D2.5mm_P7.62mm_Horizontal, symbol Device:R_Small
- added U10: 27C64, Package_DIP:DIP-28_W15.24mm, symbol Memory_EPROM:27C64
- added U2: ATTiny85, Package_DIP:DIP-8_W7.62mm, symbol MCU_Microchip_ATtiny:ATtiny13A-P
- added U3: GAL16V8, symbol Logic_Programmable:GAL16V8
- added U5: 7402, symbol 74xx:7402
- added U6: 74LS32, symbol 74xx:74LS32
- added U7: 74LS08, symbol 74xx:74LS08
- added U8: 74LS04, symbol 74xx:74LS04
- added U9: MAX232, Package_DIP:DIP-16_W7.62mm, symbol Interface_UART:MAX232
- renumbered 4MHz1 to 4MHz
Connections:
- net +5V: now also C8.1, J1.4, J3.1 (Pin_1), R3.2, R9.1, U10.27 (~{PGM}), U10.28 (VCC), U2.8 (VCC), U3.20 (VCC), U9.16 (VCC)
- net A10: now also U10.21 (A10)
- net A11: now also U10.23 (A11)
- net A12: now also U10.2 (A12)
- net A13: now also U3.19 (IO1), U8.1
- net A14: now also U3.18 (IO2), U8.5
- net A15: now also U3.17 (I03), U8.3
- net A8: now also U10.25 (A8)
- net A9: now also U10.24 (A9)
- net AD0: now also U10.11 (D0)
- net AD1: now also U10.12 (D1)
- net AD2: now also U10.13 (D2)
- net AD3: now also U10.15 (D3)
- net AD4: now also U10.16 (D4)
- net AD5: now also U10.17 (D5)
- net AD6: now also U10.18 (D6)
- net AD7: now also U10.19 (D7)
- net D1: now also J1.1
- net D2: now also J3.2 (Pin_2), U2.5 (PB0)
- net D3: now also J3.3 (Pin_3), U2.6 (PB1)
- net GND: now also J3.4 (Pin_4), U10.1 (VPP), U10.14 (GND), U2.4 (GND), U3.10 (GND)
- net Rx: now also U9.12 (R1OUT)
- net R/~{W}: now also U3.14 (IO6), U5.5
- net Tx: now also U9.11 (T1IN)
- net ~{ROM}: now also U10.22 (~{OE}), U3.12 (IO8), U5.4
- net at U4.2 (O0): now also U10.10 (A0)
- net at U4.19 (O7): now also U10.3 (A7)
- net at U4.16 (O6): now also U10.4 (A6)
- net at U4.15 (O5): now also U10.5 (A5)
- net at U4.12 (O4): now also U10.6 (A4)
- net at U4.9 (O3): now also U10.7 (A3)
- net at U4.6 (O2): now also U10.8 (A2)
- net at U4.5 (O1): now also U10.9 (A1)
- net at U1.4 (~{NMI}): now also R9.2
- net E/clk: now reaches U1.40 (E)
- net E/clk: now also U3.13 (IO7), U5.6
- net ~{IRQ}: now reaches U1.5 (~{IRQ})
- net ~{IRQ}: now also R3.1, U2.7 (PB2)
- net D0 renamed Clk-P/S2
- net Clk-P/S2: now also J1.5
- new net: U7.2, U7.4, U8.4
- new net: C11.1, U9.2 (VS+)
- new net: U7.1, U8.2
- new net: U6.1, U7.3
- new net: U6.2, U7.6
- new net: U7.5, U8.6
- new net: C7.1, U9.1 (C1+)
- new net: J2.3, U9.13 (R1IN)
- new net: J2.2, U9.14 (T1OUT)
- new net: C7.2, U9.3 (C1-)
- new net: C9.1, U9.4 (C2+)
- new net: C9.2, U9.5 (C2-)
- new net: C10.1, U9.6 (VS-)
- new net GNDREF: C10.2, C11.2, C8.2, J1.3, J1.7 (shld), J2.5, U9.15 (GND)
- new net ~{ROMce}: U10.20 (~{CE}), U3.16 (IO4), U6.3
- no-connect marks 8 -> 18
Other:
- note added: "I2C Clk"
- note added: "I2C Data"
- note added: "MCU optional: Used for ADC, Watchdog, extra timer, PWM and possibly software UART"
- note added: "PS2 Clk"
- note added: "PS2 Data"
- moved on the sheet: 4MHz, A1
